File: Main/zigduino-v6d.sch (EAGLE design)
At the start: 93 parts, among them Q1 16 MHz, SW1 EVQ-PSD02K, U1 MIC2954, U2 MIC5201-3.3YS TR, U3 ATMEGA128RFA1, U4 FT231XS-R, U6 74LVC1G17DBV, U7 MCP73831, X1 PJ002A-SMT

Commit message: -- Changed .gitignore to ignore various generated files -- Created Zigduino Micro
Parts:
- R10: PARTNO * -> ERJ-3EKF1204V
- R11: PARTNO * -> ERJ-3EKF1004V
Changed lines of the file:
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@@
 <part name="R10" library="resistor" deviceset="R-EU_" device="R0603" value="1M2">
 <attribute name="BOM" value="INCLUDE"/>
-<attribute name="PARTNO" value="*"/>
+<attribute name="PARTNO" value="ERJ-3EKF1204V"/>
 </part>
 <part name="R11" library="resistor" deviceset="R-EU_" device="R0603" value="1M">
 <attribute name="BOM" value="INCLUDE"/>
-<attribute name="PARTNO" value="*"/>
+<attribute name="PARTNO" value="ERJ-3EKF1004V"/>
 </part>
 <part name="GND18" library="supply1" deviceset="GND" device=""/>
